File: r1-rev2/pcb/echo-r1.kicad_sch (KiCad schematic)
At the start: 78 parts, among them J2 TYPE-C-31-M-12, J3 TF-115, J6 PM254-1-06-W-8.5, J7 ILI9342C, Q4 AO3401A, SW1 POWER, SW10 DPAD→, SW11 START, SW12 SELECT, SW13 VOL+, SW14 VOL-, SW2 HOLD, SW3 A, SW4 B, SW5 X, SW6 Y, SW7 DPAD↑, SW8 DPAD↓, SW9 DPAD←, U7 STM32H7R3Z8Jx, U8 W958D8NBYA5I, Y1 SC-32S32.768kHz20PPM12.5pF, Y2 XTM32024000JT00351001

Commit message: R1-Rev2: finish STM32 pin assignment and fix ERC issues
- Expanded LCD bus from 8 to 16 pins so it can be accessed by DMA2D.
- Added RDX pin to LCD bus to allow read access
- Added UART console port for easier access to debug logging
- Shorted USB HS and FS PHYs for DFU mode support
- Connected all GPIOs and peripheral pins
Parts:
- removed C25: 100 nF, Capacitor_SMD:C_0603_1608Metric, symbol Device:C_Small
- added C80: 100 nF, Capacitor_SMD:C_0402_1005Metric, symbol Device:C_Small
- added J8: Conn_01x04, symbol Connector_Generic:Conn_01x04
- added NT6, NT7: NetTie_2, echoplayer:NetTie_0.15mm_SMD, symbol Device:NetTie_2
- added R3: 68 kΩ, Resistor_SMD:R_0402_1005Metric, symbol Device:R_Small_US
Connections:
- net lcd_im0_im3 is gone; now on net lcd_im0_3: J7.30 (Pin_30)
- net lcd_mcu.cs is gone; now on net lcd.cs: U7.K11 (PD12)
- net power_vbat is gone; now on net VBAT: R12.1
- net swd_clk is gone; now on net swd.clk: U7.E10 (PA14(JTCK)
- net swd_nrst is gone; now on net swd.nrst: U7.F4 (NRST)
- net swdio is gone; now on net swd.io: J6.3 (Pin_3)
- net ~{sdmmc_pwr_en} is gone; now on net sdmmc_pwr_en: Q4.1 (G), R25.2
- net +3V3: now also J8.4 (Pin_4)
- net GND: now also J7.7 (Pin_7), C80.2, J8.2 (Pin_2), R3.2
- net VBUS: now also U7.C7 (PM14)
- net adc_vbat: now also U7.K4 (PA7)
- net adc_vbus: now also U7.M3 (PC5)
- net backlight_pwm: now also U7.L12 (PD13)
- net boot0: now also R3.1
- net button_a: now also U7.K2 (PA3)
- net button_b: now also U7.L2 (PA4)
- net button_down: now also U7.B12 (PD4)
- net button_hold: now also U7.G3 (PC0)
- net button_left: now also U7.B6 (PD5)
- net button_power: now also U7.E8 (PM0)
- net button_right: now also U7.C6 (PD6)
- net button_select: now also U7.L11 (PD11)
- net button_start: now also U7.M11 (PD10)
- net button_up: now also U7.D10 (PD3)
- net button_vol+: now also U7.A5 (PD7)
- net button_vol-: now also U7.J8 (PD8)
- net button_x: now also U7.J4 (PA5)
- net button_y: now also U7.M2 (PA6)
- net cpu_power_on: now also U7.H11 (PD14)
- net hp_micbutton+: now also U7.J1 (PC2)
- net hp_micbutton-: now also U7.H2 (PC3)
- net lcd_im1: now also U7.L4 (PB0)
- net lcd_reset: now also U7.C3 (PB9)
- net sdmmc_detect: now also U7.B4 (PE0)
- net usb_d+: now also NT7.1
- net usb_d-: now also NT6.1
- net vfbsmps: now also C80.1
- net xspi_reset: now also U7.J6 (PO1)
- net lcd.rdx: now reaches J7.12 (Pin_12)
- net lcd.rdx: now also U7.M4 (PB1)
- net lcd.d8: now reaches J7.21 (Pin_21)
- net lcd.d8: now also U7.J11 (PB13)
- net lcd.d9: now reaches J7.22 (Pin_22)
- net lcd.d9: now also U7.H10 (PB12)
- net lcd.d10: now reaches J7.23 (Pin_23)
- net lcd.d10: now also U7.K12 (PB11)
- net lcd.d11: now reaches J7.24 (Pin_24)
- net lcd.d11: now also U7.J10 (PB10)
- net lcd.d12: now reaches J7.25 (Pin_25)
- net lcd.d12: now also U7.A4 (PB5)
- net lcd.d13: now reaches J7.26 (Pin_26)
- net lcd.d13: now also U7.C5 (PB4(NJTRST))
- net lcd.d14: now reaches J7.27 (Pin_27)
- net lcd.d14: now also U7.B5 (PB3(JTDO)
- net lcd.d15: now reaches J7.28 (Pin_28)
- net lcd.d15: now also U7.D12 (PA15(JTDI))
- net lcd_im0_3: now reaches U7.A3 (PB6)
- net usb_fs_d+: now reaches U7.A7 (PM11)
- net usb_fs_d+: now also NT7.2
- net codec_dvdd_en: now reaches U7.B10 (PM2)
- net codec_reset: now reaches U7.B11 (PM3)
- net sdmmc_pwr_en: now reaches U7.B3 (PE1)
- net usb_fs_d-: now reaches U7.B7 (PM12)
- net usb_fs_d-: now also NT6.2
- net codec_avdd_en: now reaches U7.C10 (PM1)
- net chg_enable: now reaches U7.G9 (PC7)
- net chg_charging: now reaches U7.H12 (PC6)
- net uart_tx: now reaches U7.H9 (PB14)
- net uart_tx: now also J8.1 (Pin_1)
- net uart_rx: now reaches U7.J12 (PB15)
- net uart_rx: now also J8.3 (Pin_3)
- net lo_detect: now reaches U7.L3 (PC4)
- net nrst renamed swd.nrst
- net swclk renamed swd.clk
- net swd_io renamed swd.io
- now unconnected: U8.A5 (RFU), U8.B5 (RFU), U8.C2 (RFU), U8.C5 (RFU)
- no-connect marks 20 -> 12
Other:
- note added: "DVDD"
- note added: "SERIAL CONSOLE"
- note added: "TE pin"
- note removed: "DB8-DB15 unused"
- moved on the sheet: C32, C42, C56, C57, C58, C59, C60, C68, C69, C70, C71, C73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
