File: r1-rev1/echo-r1-rev1.kicad_pcb (KiCad board)
At the start: 6 copper layers, 55 x 95 mm, 154 parts, among them J1 GT-BTP30003-xxxA-16A, J2 TYPE-C-31-M-12, J3 TF-115, J4 HP_3.5mm, J5 LO_3.5mm, J6 AFD01-S35FCC-00, J7 PM254-1-06-W-8.5, Q2 AO3401A, Q5 AO3401A, Q6 AO3401A, Q7 AO3401A, SW1 DPAD↑, SW10 X, SW11 Y, SW12 START, SW13 SELECT, SW14 HOLD, SW2 DPAD↓, SW3 DPAD←, SW4 DPAD→, SW5 A, SW6 B, SW7 VOL+, SW8 VOL-, SW9 POWER, U1 LM66100DCK, U10 SY7200A, U2 TPS62A01DRLR, U3 TPS62A01DRLR, U4 XC6206P33xMR, U5 TP4057, U6 STM32H743IGTx, U7 W9825G6KH-x, U8 USB3320C-EZK, U9 TLV320AIC3104, Y1 SC-32S32.768kHz20PPM12.5pF, Y2 XTM32024000JT00351001

Commit message: Fix incorrect 3.5mm jack pinout
Document the R1-Rev1's wrong pinout properly and fix the pinout
in later revs so that jacks will work properly without needing
a custom adapter.

See Github issue: #12
Connections:
- J4 pad R1: /audio/hp_right -> /audio/hp_left
- J4 pad R2: /audio/hp_com -> /audio/hp_right
- J4 pad T: /audio/hp_left -> /audio/hp_com
- J5 pad R1: Net-(D5-IO1) -> Net-(D5-IO2)
- J5 pad R2: GND -> Net-(D5-IO1)
- J5 pad T: Net-(D5-IO2) -> GND
Changed lines of the file:
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@@
 			(size 1.05 0.7)
 			(layers "B.Cu" "B.Mask" "B.Paste")
-			(net 51 "unconnected-(SW14-PadMP)_1")
+			(net 52 "unconnected-(SW14-PadMP)_2")
 			(pinfunction "MP")
 			(pintype "passive+no_connect")
@@
 			(size 1.05 0.7)
 			(layers "B.Cu" "B.Mask" "B.Paste")
-			(net 50 "unconnected-(SW14-PadMP)")
+			(net 51 "unconnected-(SW14-PadMP)_1")
 			(pinfunction "MP")
 			(pintype "passive+no_connect")
@@
 			(size 1.05 0.7)
 			(layers "B.Cu" "B.Mask" "B.Paste")
-			(net 52 "unconnected-(SW14-PadMP)_2")
+			(net 50 "unconnected-(SW14-PadMP)")
 			(pinfunction "MP")
 			(pintype "passive+no_connect")
@@
 			(size 1.05 0.7)
 			(layers "B.Cu" "B.Mask" "B.Paste")
-			(net 40 "unconnected-(SW7-B-PadMP)_1")
+			(net 200 "unconnected-(SW7-B-PadMP)_3")
 			(pinfunction "B")
 			(pintype "passive+no_connect")
@@
 			(size 0.65 1.3)
 			(layers "B.Cu" "B.Mask" "B.Paste")
-			(net 200 "unconnected-(SW7-B-PadMP)_3")
+			(net 40 "unconnected-(SW7-B-PadMP)_1")
 			(pinfunction "B")
 			(pintype "passive+no_connect")
@@
 		)
 		(pad "R1" thru_hole oval
-			(at -1.8 2.25 90)
+			(at 1.3 2.25 90)
 			(size 2 1)
 			(drill oval 1.5 0.5)
 			(layers "*.Cu" "*.Mask")
 			(remove_unused_layers no)
-			(net 73 "/audio/hp_right")
+			(net 72 "/audio/hp_left")
 			(pintype "passive")
 		)
 		(pad "R2" thru_hole oval
-			(at 5.4 2.25 90)
+			(at -1.8 2.25 90)
 			(size 2 1)
 			(drill oval 1.5 0.5)
 			(layers "*.Cu" "*.Mask")
 			(remove_unused_layers no)
-			(net 74 "/audio/hp_com")
+			(net 73 "/audio/hp_right")
 			(pintype "passive")
 		)
@@
 		)
 		(pad "T" thru_hole oval
-			(at 1.3 2.25 90)
+			(at 5.4 2.25 90)
 			(size 2 1)
 			(drill oval 1.5 0.5)
 			(layers "*.Cu" "*.Mask")
 			(remove_unused_layers no)
-			(net 72 "/audio/hp_left")
+			(net 74 "/audio/hp_com")
 			(pintype "passive")
 		)
@@
 			(size 0.65 1.3)
 			(layers "B.Cu" "B.Mask" "B.Paste")
-			(net 46 "unconnected-(SW9-B-PadMP)")
+			(net 202 "unconnected-(SW9-B-PadMP)_3")
 			(pinfunction "B")
 			(pintype "passive+no_connect")
@@
 			(size 1.05 0.7)
 			(layers "B.Cu" "B.Mask" "B.Paste")
-			(net 47 "unconnected-(SW9-B-PadMP)_1")
+			(net 46 "unconnected-(SW9-B-PadMP)")
 			(pinfunction "B")
 			(pintype "passive+no_connect")
@@
 			(size 1.05 0.7)
 			(layers "B.Cu" "B.Mask" "B.Paste")
-			(net 48 "unconnected-(SW9-B-PadMP)_2")
+			(net 47 "unconnected-(SW9-B-PadMP)_1")
 			(pinfunction "B")
 			(pintype "passive+no_connect")
@@
 			(size 0.65 1.3)
 			(layers "B.Cu" "B.Mask" "B.Paste")
-			(net 202 "unconnected-(SW9-B-PadMP)_3")
+			(net 48 "unconnected-(SW9-B-PadMP)_2")
 			(pinfunction "B")
 			(pintype "passive+no_connect")
@@
 		)
 		(pad "R1" thru_hole oval
-			(at -1.8 2.25 90)
+			(at 1.3 2.25 90)
 			(size 2 1)
 			(drill oval 1.5 0.5)
 			(layers "*.Cu" "*.Mask")
 			(remove_unused_layers no)
-			(net 11 "Net-(D5-IO1)")
+			(net 10 "Net-(D5-IO2)")
 			(pintype "passive")
 		)
 		(pad "R2" thru_hole oval
-			(at 5.4 2.25 90)
+			(at -1.8 2.25 90)
 			(size 2 1)
 			(drill oval 1.5 0.5)
 			(layers "*.Cu" "*.Mask")
 			(remove_unused_layers no)
-			(net 1 "GND")
+			(net 11 "Net-(D5-IO1)")
 			(pintype "passive")
 		)
@@
 		)
 		(pad "T" thru_hole oval
-			(at 1.3 2.25 90)
+			(at 5.4 2.25 90)
 			(size 2 1)
 			(drill oval 1.5 0.5)
 			(layers "*.Cu" "*.Mask")
 			(remove_unused_layers no)
-			(net 10 "Net-(D5-IO2)")
+			(net 1 "GND")
 			(pintype "passive")
 		)
